Commit message: 更新Gazebo和正对目标改为树冠

File: urdf/tracked_canopy_robot.urdf.xacro (robot description, xacro)
@@ -1,4 +1,6 @@
 <?xml version="1.0"?>
 <robot name="tracked_canopy_robot" xmlns:xacro="http://www.ros.org/wiki/xacro">
+  <!-- Gazebo 中是否显示全部激光射线；只影响显示，不影响 /scan_2d。 -->
+  <xacro:arg name="visualize_laser" default="false"/>
   <!--
     tracked_canopy_robot.urdf.xacro
@@ -6,5 +8,5 @@
     建模策略：
       - 外观看起来像履带底盘；
-      - 运动学上先用差速小车插件 gazebo_ros_diff_drive；
+      - 运动学使用 Gazebo 平面运动插件；
       - 这样你可以先验证 /cmd_vel、/Odometry、/scan_2d 和控制节点闭环；
       - 后续再升级成更复杂的履带接触物理模型。
@@ -15,13 +17,16 @@
       - 雷达安装在车体右侧，朝右看树冠，所以相对 base_link 绕 z 轴旋转 -90 度。
   -->
-  <!-- 常用尺寸参数，后续要改车体尺寸主要改这里。 -->
-  <xacro:property name="base_length" value="0.80"/>
-  <xacro:property name="base_width" value="0.55"/>
-  <xacro:property name="base_height" value="0.22"/>
-  <xacro:property name="track_length" value="0.86"/>
+  <!--
+    实车俯视外形约 1.60 m × 1.00 m。base_width 不含履带，左右履带
+    加入后总宽度为 0.76 + 2 × 0.12 = 1.00 m。
+  -->
+  <xacro:property name="base_length" value="1.50"/>
+  <xacro:property name="base_width" value="0.76"/>
+  <xacro:property name="base_height" value="0.34"/>
+  <xacro:property name="track_length" value="1.60"/>
   <xacro:property name="track_width" value="0.12"/>
-  <xacro:property name="track_height" value="0.16"/>
-  <xacro:property name="wheel_radius" value="0.08"/>
-  <xacro:property name="wheel_width" value="0.05"/>
+  <xacro:property name="track_height" value="0.24"/>
+  <xacro:property name="wheel_radius" value="0.16"/>
+  <xacro:property name="wheel_width" value="0.08"/>
   <!-- base_footprint 是地面投影坐标系，常用于导航。 -->
   <link name="base_footprint"/>
@@ -47,12 +52,6 @@
       </material>
     </visual>
-    <collision>
-      <origin xyz="0 0 0"/>
-      <geometry>
-        <box size="${base_length} ${base_width} ${base_height}"/>
-      </geometry>
-    </collision>
   </link>
-  <!-- 左右履带只是视觉和碰撞外壳，真实驱动由四个轮子和差速插件负责。 -->
+  <!-- 左右履带是不参与地面碰撞的视觉外壳。 -->
   <link name="left_track_link">
     <visual>
@@ -65,10 +64,4 @@
       </material>
     </visual>
-    <collision>
-      <origin xyz="0 0 0"/>
-      <geometry>
-        <box size="${track_length} ${track_width} ${track_height}"/>
-      </geometry>
-    </collision>
   </link>
   <joint name="left_track_fixed" type="fixed">
@@ -85,10 +78,4 @@
       <material name="track_dark"/>
     </visual>
-    <collision>
-      <origin xyz="0 0 0"/>
-      <geometry>
-        <box size="${track_length} ${track_width} ${track_height}"/>
-      </geometry>
-    </collision>
   </link>
   <joint name="right_track_fixed" type="fixed">
@@ -97,10 +84,6 @@
     <origin xyz="0 ${-(base_width / 2.0 + track_width / 2.0)} ${-base_height / 2.0 + track_height / 2.0}" rpy="0 0 0"/>
   </joint>
-  <!--
-    四个驱动轮。
-    Gazebo 的 diff_drive 插件需要左轮 joint 和右轮 joint。
-    这里用前方两个轮子做插件驱动轮，后方两个轮子作为自由支撑轮。
-  -->
-  <xacro:macro name="drive_wheel" params="prefix x y driven">
+  <!-- 四个车轮仅用于外形显示，固定在车体上以避免自由关节抖动。 -->
+  <xacro:macro name="display_wheel" params="prefix x y">
     <link name="${prefix}_wheel_link">
       <inertial>
@@ -118,22 +101,15 @@
         </material>
       </visual>
-      <collision>
-        <origin xyz="0 0 0" rpy="1.57079632679 0 0"/>
-        <geometry>
-          <cylinder radius="${wheel_radius}" length="${wheel_width}"/>
-        </geometry>
-      </collision>
     </link>
-    <joint name="${prefix}_wheel_joint" type="continuous">
+    <joint name="${prefix}_wheel_joint" type="fixed">
       <parent link="base_link"/>
       <child link="${prefix}_wheel_link"/>
-      <origin xyz="${x} ${y} ${-base_height / 2.0}" rpy="0 0 0"/>
-      <axis xyz="0 1 0"/>
+      <origin xyz="${x} ${y} ${-base_height / 2.0 + wheel_radius}" rpy="0 0 0"/>
     </joint>
   </xacro:macro>
-  <xacro:drive_wheel prefix="front_left"  x="0.28"  y="${base_width / 2.0 + track_width / 2.0}" driven="true"/>
-  <xacro:drive_wheel prefix="front_right" x="0.28"  y="${-(base_width / 2.0 + track_width / 2.0)}" driven="true"/>
-  <xacro:drive_wheel prefix="rear_left"   x="-0.28" y="${base_width / 2.0 + track_width / 2.0}" driven="false"/>
-  <xacro:drive_wheel prefix="rear_right"  x="-0.28" y="${-(base_width / 2.0 + track_width / 2.0)}" driven="false"/>
+  <xacro:display_wheel prefix="front_left"  x="0.55"  y="${base_width / 2.0 + track_width / 2.0}"/>
+  <xacro:display_wheel prefix="front_right" x="0.55"  y="${-(base_width / 2.0 + track_width / 2.0)}"/>
+  <xacro:display_wheel prefix="rear_left"   x="-0.55" y="${base_width / 2.0 + track_width / 2.0}"/>
+  <xacro:display_wheel prefix="rear_right"  x="-0.55" y="${-(base_width / 2.0 + track_width / 2.0)}"/>
   <!-- 雷达安装架。雷达在右侧，朝向右侧树冠。 -->
   <link name="livox_frame">
@@ -147,34 +123,33 @@
       </material>
     </visual>
-    <collision>
-      <origin xyz="0 0 0"/>
-      <geometry>
-        <box size="0.10 0.08 0.08"/>
-      </geometry>
-    </collision>
   </link>
   <joint name="livox_joint" type="fixed">
     <parent link="base_link"/>
     <child link="livox_frame"/>
-    <origin xyz="0.05 -0.36 0.10" rpy="0 0 -1.57079632679"/>
+    <origin xyz="0.00 -0.50 0.20" rpy="0 0 -1.57079632679"/>
   </joint>
-  <!-- Gazebo 差速驱动插件。它订阅 /cmd_vel，发布 /Odometry。 -->
+  <!--
+    机器人是平面运动学模型：所有外形都会合并到 base_footprint，
+    关闭根链接重力可防止没有承重碰撞体的车辆穿过地面。
+  -->
+  <gazebo reference="base_footprint">
+    <gravity>false</gravity>
+  </gazebo>
+  <!--
+    这一阶段主要验证树冠跟随状态机，因此用平面运动插件精确执行
+    /cmd_vel，并发布 /Odometry。这可以避免 Gazebo 轮胎摩擦参数导致的
+    履带侧滑偏差；车体、履带和车轮仍按实际尺寸显示，但不参与地面碰撞。
+  -->
   <gazebo>
-    <plugin name="tracked_diff_drive" filename="libgazebo_ros_diff_drive.so">
-      <rosDebugLevel>na</rosDebugLevel>
-      <publishWheelTF>false</publishWheelTF>
-      <publishWheelJointState>true</publishWheelJointState>
+    <plugin name="tracked_planar_drive" filename="libgazebo_ros_planar_move.so">
       <alwaysOn>true</alwaysOn>
       <updateRate>50.0</updateRate>
-      <leftJoint>front_left_wheel_joint</leftJoint>
-      <rightJoint>front_right_wheel_joint</rightJoint>
-      <wheelSeparation>${base_width + track_width}</wheelSeparation>
-      <wheelDiameter>${2.0 * wheel_radius}</wheelDiameter>
-      <torque>20</torque>
+      <odometryRate>50.0</odometryRate>
+      <cmdTimeout>0.5</cmdTimeout>
       <commandTopic>/cmd_vel</commandTopic>
       <odometryTopic>/Odometry</odometryTopic>
       <odometryFrame>odom</odometryFrame>
       <robotBaseFrame>base_link</robotBaseFrame>
-      <publishOdomTF>true</publishOdomTF>
+      <broadcastTF>true</broadcastTF>
     </plugin>
   </gazebo>
@@ -183,18 +158,18 @@
     <sensor name="side_lidar" type="ray">
       <always_on>true</always_on>
-      <visualize>true</visualize>
-      <update_rate>15</update_rate>
+      <visualize>$(arg visualize_laser)</visualize>
+      <update_rate>10</update_rate>
       <ray>
         <scan>
           <horizontal>
-            <samples>720</samples>
+            <samples>1800</samples>
             <resolution>1</resolution>
-            <min_angle>-2.09439510239</min_angle>
-            <max_angle>2.09439510239</max_angle>
+            <min_angle>-3.14159265359</min_angle>
+            <max_angle>3.14159265359</max_angle>
           </horizontal>
         </scan>
         <range>
-          <min>0.20</min>
-          <max>4.00</max>
+          <min>0.10</min>
+          <max>50.00</max>
           <resolution>0.01</resolution>
         </range>
